Commit message: Chnages with the Probe Link origins, inertial matrix and other enhancements

File: robot_simulation/URDF/sr_scara_hx.urdf (robot description, URDF)
Before this commit: robot sr_scara_hx, 6 links, 5 joints
Links:
- link base_link: mass 1.0 -> 30.0
- link gripper_end_effector: mass 0.3 -> 0.1
- link link1: mass 1.0 -> 10.0
- link link2: mass 1.0 -> 10.0
- link probe: mass 1.0 -> 2.0
Joints:
- joint joint1: limit lower=-2.617 upper=2.617 effort=3.0 velocity=0.01 -> lower=-2.792 upper=2.792 effort=3.0 velocity=0.01
- joint joint2: limit lower=-2.617 upper=2.617 effort=3.0 velocity=0.01 -> lower=-2.443 upper=2.443 effort=3.0 velocity=0.01
- joint joint3: limit lower=-0.1 upper=0.05 effort=3.0 velocity=0.01 -> lower=0.0 upper=0.13 effort=3.0 velocity=0.01
- joint joint4: origin xyz=-0.65 0 0.26 rpy=0 0 0 -> xyz=-0.65 0 0.158 rpy=0 0 0

File: robot_simulation/URDF/sr_scara_hx.xacro (robot description, xacro)
@@ -27,5 +27,5 @@
  <inertial>
       <origin xyz="0 0 0.00158925" rpy="0 0 0"/>
-      <mass value="1.0"/>
+      <mass value="30.0"/>
       <inertia
 	  ixx="1.0" ixy="0.0" ixz="0.0"
@@ -50,5 +50,5 @@
  <inertial>
       <origin xyz="0 0 0" rpy="0 0 0"/>
-      <mass value="1.0"/>
+      <mass value="10.0"/>
       <inertia
 	  ixx="1.0" ixy="0.0" ixz="0.0"
@@ -73,5 +73,5 @@
  <inertial>
       <origin xyz="0.300 0 0" rpy="0 0 0"/>
-      <mass value="1.0"/>
+      <mass value="10.0"/>
       <inertia
 	  ixx="1.0" ixy="0.0" ixz="0.0"
@@ -82,5 +82,5 @@
 <link name="probe">
  <visual>
-  <origin xyz="0 0 0" rpy="0 0 0" />
+  <origin xyz="-0.65 0 0.43" rpy="0 0 0" />
   <geometry>
      <mesh filename="package://robot_simulation/meshes/End_link_R01.stl" scale="0.001 0.001 0.001"/>
@@ -89,5 +89,5 @@
  </visual>
  <collision>
-  <origin xyz="0 0 0" rpy="0 0 0" />
+  <origin xyz="-0.65 0 0.43" rpy="0 0 0" />
   <geometry>
      <mesh filename="package://robot_simulation/meshes/End_link_R01.stl" scale="0.001 0.001 0.001"/>
@@ -95,6 +95,6 @@
  </collision>
  <inertial>
-      <origin xyz="0 0 0" rpy="0 0 0"/>
-      <mass value="1.0"/>
+      <origin xyz="-0.65 0 0.43" rpy="0 0 0"/>
+      <mass value="2.0"/>
       <inertia
 	  ixx="1.0" ixy="0.0" ixz="0.0"
@@ -121,6 +121,6 @@
      <mass value="0.3"/>
      <inertia
-         ixx="1.0" ixy="1.0" ixz="1.0"
-	 iyy="1.0" iyz="1.0"
+         ixx="1.0" ixy="0.0" ixz="0.0"
+	 iyy="1.0" iyz="0.0"
 	 izz="1.0"/>
  </inertial>
@@ -142,8 +142,8 @@
  <inertial>
      <origin xyz="0 0 0" rpy="0 0 0"/>
-     <mass value="0.3"/>
+     <mass value="0.1"/>
      <inertia
-         ixx="1.0" ixy="1.0" ixz="1.0"
-	 iyy="1.0" iyz="1.0"
+         ixx="1.0" ixy="0.0" ixz="0.0"
+	 iyy="1.0" iyz="0.0"
 	 izz="1.0"/>
  </inertial>
@@ -152,5 +152,5 @@
 <joint name="joint1" type="revolute">
   <axis xyz="0 0 1" />
-  <limit effort="3.0" velocity="0.01" lower="-2.617" upper="2.617"/>
+  <limit effort="3.0" velocity="0.01" lower="-2.792" upper="2.792"/>
   <origin xyz="0 0 0.00158925" rpy="0 0 0" />
   <parent link="base_link" />
@@ -159,5 +159,5 @@
 <joint name="joint2" type="revolute">
  <axis xyz="0 0 1" />
- <limit effort="3.0" velocity="0.01" lower="-2.617" upper="2.617"/>
+ <limit effort="3.0" velocity="0.01" lower="-2.443" upper="2.443"/>
  <origin xyz="-0.3 0 0" rpy="0 0 0" />
  <parent link="link1" />
@@ -166,5 +166,5 @@
 <joint name="joint3" type="prismatic">
  <axis xyz="0 0 1" />
- <limit effort="3.0" velocity="0.01" lower="-0.1" upper="0.05"/>
+ <limit effort="3.0" velocity="0.01" lower="0.0" upper="0.13"/>
  <origin xyz="0.3 0 0" rpy="0 0 0" />
  <parent link="link2" />
@@ -172,5 +172,5 @@
 </joint>
 <joint name ="joint4" type="fixed">
- <origin xyz="-0.65 0 0.26" rpy="0 0 0"/>
+ <origin xyz="-0.65 0 0.158" rpy="0 0 0"/>
  <parent link = "probe"/>
  <child link = "gripper"/>
