Commit message: Closure

File: sr_scara_hx_description/URDF/sr_scara_hx.urdf (robot description, URDF)
Before this commit: robot sr_scara_hx, 6 links, 5 joints
Joints:
- joint joint1: origin xyz=0 0 0.00158925 rpy=0 0 0 -> xyz=0 0 0.33 rpy=0 0 0
- joint joint2: origin xyz=-0.3 0 0 rpy=0 0 0 -> xyz=-0.35 0 0.08 rpy=0 0 0
- joint joint3: origin xyz=0.3 0 0 rpy=0 0 0 -> xyz=-0.38 0 0.08 rpy=0 0 0
- joint joint4: origin xyz=-0.65 0 0.158 rpy=0 0 0 -> xyz=0 0 -0.335 rpy=0 0 0

File: sr_scara_hx_description/URDF/sr_scara_hx.xacro (robot description, xacro)
@@ -13,5 +13,5 @@
 <link name="base_link">
  <visual>
-  <origin xyz="0 0 0.00158925" rpy="0 0 0" />
+  <origin xyz="0 0 0.15" rpy="0 0 0" />
    <geometry>
      <mesh filename="package://robot_simulation/meshes/base_R01.stl" scale="0.001 0.001 0.001"/>
@@ -20,5 +20,5 @@
  </visual>
  <collision>
-  <origin xyz="0 0 0.00158925" rpy="0 0 0" />
+  <origin xyz="0 0 0.15" rpy="0 0 0" />
    <geometry>
      <mesh filename="package://robot_simulation/meshes/base_R01.stl" scale="0.001 0.001 0.001"/>
@@ -26,5 +26,5 @@
  </collision>
  <inertial>
-      <origin xyz="0 0 0.00158925" rpy="0 0 0"/>
+      <origin xyz="0 0 0.15" rpy="0 0 0"/>
       <mass value="3000.0"/>
       <inertia
@@ -36,5 +36,5 @@
 <link name="link1">
  <visual>
-  <origin xyz="0 0 0" rpy="0 0 0" />
+  <origin xyz="-0.18 0 0.03" rpy="0 0 0" />
    <geometry>
      <mesh filename="package://robot_simulation/meshes/arm_link_R01.stl" scale="0.001 0.001 0.001"/>
@@ -43,5 +43,5 @@
  </visual>
  <collision>
-  <origin xyz="0 0 0" rpy="0 0 0" />
+  <origin xyz="-0.18 0 0.03" rpy="0 0 0" />
    <geometry>
      <mesh filename="package://robot_simulation/meshes/arm_link_R01.stl" scale="0.001 0.001 0.001"/>
@@ -49,5 +49,5 @@
  </collision>
  <inertial>
-      <origin xyz="0 0 0" rpy="0 0 0"/>
+      <origin xyz="-0.18 0 0.03" rpy="0 0 0"/>
       <mass value="10.0"/>
       <inertia
@@ -59,5 +59,5 @@
 <link name="link2">
  <visual>
-  <origin xyz="0.300 0 0" rpy="0 0 0" />
+  <origin xyz="-0.23 0 0.06" rpy="0 0 0" />
    <geometry>
      <mesh filename="package://robot_simulation/meshes/head_link_R01.stl" scale="0.001 0.001 0.001"/>
@@ -66,5 +66,5 @@
  </visual>
  <collision>
-  <origin xyz="0.300 0 0" rpy="0 0 0" />
+  <origin xyz="-0.23 0 0.06" rpy="0 0 0" />
    <geometry>
      <mesh filename="package://robot_simulation/meshes/head_link_R01.stl" scale="0.001 0.001 0.001"/>
@@ -72,5 +72,5 @@
   </collision>
  <inertial>
-      <origin xyz="0.300 0 0" rpy="0 0 0"/>
+      <origin xyz="-0.23 0 0.06" rpy="0 0 0"/>
       <mass value="10.0"/>
       <inertia
@@ -82,5 +82,5 @@
 <link name="probe">
  <visual>
-  <origin xyz="-0.65 0 0.43" rpy="0 0 0" />
+  <origin xyz="0 0 -0.062" rpy="0 0 0" />
   <geometry>
      <mesh filename="package://robot_simulation/meshes/End_link_R01.stl" scale="0.001 0.001 0.001"/>
@@ -89,5 +89,5 @@
  </visual>
  <collision>
-  <origin xyz="-0.65 0 0.43" rpy="0 0 0" />
+  <origin xyz="0 0 -0.062" rpy="0 0 0" />
   <geometry>
      <mesh filename="package://robot_simulation/meshes/End_link_R01.stl" scale="0.001 0.001 0.001"/>
@@ -95,5 +95,5 @@
  </collision>
  <inertial>
-      <origin xyz="-0.65 0 0.43" rpy="0 0 0"/>
+      <origin xyz="0 0 -0.062" rpy="0 0 0"/>
       <mass value="2.0"/>
       <inertia
@@ -153,5 +153,5 @@
   <axis xyz="0 0 1" />
   <limit effort="3.0" velocity="0.01" lower="-2.792" upper="2.792"/>
-  <origin xyz="0 0 0.00158925" rpy="0 0 0" />
+  <origin xyz="0 0 0.33" rpy="0 0 0" />
   <parent link="base_link" />
   <child link="link1" />
@@ -160,5 +160,5 @@
  <axis xyz="0 0 1" />
  <limit effort="3.0" velocity="0.01" lower="-2.443" upper="2.443"/>
- <origin xyz="-0.3 0 0" rpy="0 0 0" />
+ <origin xyz="-0.35 0 0.08" rpy="0 0 0" />
  <parent link="link1" />
  <child link="link2" />
@@ -167,10 +167,10 @@
  <axis xyz="0 0 1" />
  <limit effort="3.0" velocity="0.01" lower="0.0" upper="0.13"/>
- <origin xyz="0.3 0 0" rpy="0 0 0" />
+ <origin xyz="-0.38 0 0.08" rpy="0 0 0" />
  <parent link="link2" />
  <child link="probe" />
 </joint>
 <joint name ="joint4" type="fixed">
- <origin xyz="-0.65 0 0.158" rpy="0 0 0"/>
+ <origin xyz="0 0 -0.335" rpy="0 0 0"/>
  <parent link = "probe"/>
  <child link = "gripper"/>
@@ -185,8 +185,8 @@
   <type>transmission_interface/SimpleTransmission</type>
     <joint name="joint1">
-      <hardwareInterface>PositionJointInterface</hardwareInterface>
+      <hardwareInterface>hardware_interface/PositionJointInterface</hardwareInterface>
     </joint>
     <actuator name="motor1">
-      <hardwareInterface>PositionJointInterface</hardwareInterface>
+      <hardwareInterface>hardware_interface/PositionJointInterface</hardwareInterface>
       <mechanicalReduction>1</mechanicalReduction>
     </actuator>
@@ -195,8 +195,8 @@
    <type>transmission_interface/SimpleTransmission</type>
     <joint name="joint2">
-      <hardwareInterface>PositionJointInterface</hardwareInterface>
+      <hardwareInterface>hardware_interface/PositionJointInterface</hardwareInterface>
     </joint>
     <actuator name="motor2">
-      <hardwareInterface>PositionJointInterface</hardwareInterface>
+      <hardwareInterface>hardware_interface/PositionJointInterface</hardwareInterface>
       <mechanicalReduction>1</mechanicalReduction>
     </actuator>
@@ -205,8 +205,8 @@
    <type>transmission_interface/SimpleTransmission</type>
     <joint name="joint3">
-      <hardwareInterface>PositionJointInterface</hardwareInterface>
+      <hardwareInterface>hardware_interface/PositionJointInterface</hardwareInterface>
     </joint>
     <actuator name="motor3">
-      <hardwareInterface>PositionJointInterface</hardwareInterface>
+      <hardwareInterface>hardware_interface/PositionJointInterface</hardwareInterface>
       <mechanicalReduction>1</mechanicalReduction>
     </actuator>
